File: Eletrônica/Toggle/Toggle.brd (EAGLE design)
At the start: 15.2 x 15.2 mm, 17 parts, among them Q2 MOSFET-NCHANNELBSS123LT1G, Q3 MOSFET-NCHANNELBSS123LT1G

Commit message: Eagle .gitignore updates
Parts:
- removed Q3: MOSFET-NCHANNELBSS123LT1G, SparkFun-DiscreteSemi:SOT23
- removed Q4: (no value), transistor-power:MICRO3
- R2, R4: value 100k -> 1M
- moved R4 16.3 mm to (0.00, -6.35), turned to 0 degrees
Connections:
- removed net N$45: D1.C, Q3.3, R2.1, R3.2
- net ARD_OFF: now also D1.C, R2.1, R3.2; no longer Q3.1, Q4.1, R4.1
- net GND: now also R4.1; no longer Q3.2, Q4.2, R4.2
- net N$2: now also R4.2
Routing:
- net N$45: track 8.14 -> 0.00 mm
- net ARD_OFF: track 7.77 -> 12.5 mm
Changed lines of the file:
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@@
 <attribute name="NAME" x="5.87375" y="12.3825" size="0.762" layer="25" font="vector" ratio="15"/>
 </element>
-<element name="R2" library="wes" package="R0603" value="100k" x="4.1275" y="7.3025" smashed="yes" rot="R90">
+<element name="R2" library="wes" package="R0603" value="1M" x="4.1275" y="7.3025" smashed="yes" rot="R90">
 <attribute name="NAME" x="3.4925" y="5.08" size="0.762" layer="25" font="vector" ratio="15"/>
 </element>
@@
 </element>
 <element name="BUT" library="SparkFun-Connectors" package="1X02_NO_SILK" value="M021X02_NO_SILK" x="11.43" y="13.97" smashed="yes"/>
-<element name="Q3" library="SparkFun-DiscreteSemi" package="SOT23" value="MOSFET-NCHANNELBSS123LT1G" x="10.16" y="2.54" smashed="yes" rot="R90">
-<attribute name="PROD_ID" value="TRANS-08345" x="10.16" y="2.54" size="1.778" layer="27" rot="R90" display="off"/>
-<attribute name="NAME" x="9.30275" y="1.61925" size="0.762" layer="25" ratio="15" rot="R180"/>
-</element>
-<element name="R4" library="wes" package="R0603" value="100k" x="13.6525" y="2.54" smashed="yes" rot="R90">
-<attribute name="NAME" x="13.0175" y="4.1275" size="0.762" layer="25" font="vector" ratio="15"/>
-</element>
 <element name="R5" library="wes" package="R0603" value="10k" x="13.6525" y="10.4775" smashed="yes" rot="R90">
 <attribute name="NAME" x="13.0175" y="11.90625" size="0.762" layer="25" font="vector" ratio="15"/>
@@
 <attribute name="VALUE" x="8.2931" y="6.6167" size="0.4064" layer="27" rot="R90"/>
 </element>
-<element name="Q4" library="transistor-power" package="MICRO3" value="" x="10.16" y="-2.54" rot="R90"/>
+<element name="R4" library="wes" package="R0603" value="1M" x="0" y="-6.35"/>
 </elements>
 <signals>
@@
 <signal name="ARD_OFF">
 <contactref element="JP3" pad="3"/>
-<contactref element="Q3" pad="1"/>
-<contactref element="R4" pad="1"/>
-<wire x1="11.26" y1="1.59" x2="13.745" y2="1.59" width="0.2032" layer="1"/>
-<wire x1="13.745" y1="1.59" x2="13.6525" y2="1.815" width="0.2032" layer="1"/>
 <wire x1="6.35" y1="1.27" x2="10.94" y2="1.27" width="0.2032" layer="1"/>
-<wire x1="10.94" y1="1.27" x2="11.26" y2="1.59" width="0.2032" layer="1"/>
-<contactref element="Q4" pad="1"/>
-<wire x1="6.35" y1="1.27" x2="11.16" y2="-3.49" width="0" layer="19" extent="1-1"/>
+<contactref element="R3" pad="2"/>
+<contactref element="R2" pad="1"/>
+<wire x1="4.1275" y1="6.5775" x2="5.715" y2="6.5775" width="0.2032" layer="1"/>
+<wire x1="8.89" y1="4.1275" x2="8.89" y2="2.71" width="0.2032" layer="1"/>
+<wire x1="8.89" y1="4.1275" x2="6.82625" y2="6.19125" width="0.2032" layer="1"/>
+<wire x1="6.82625" y1="6.19125" x2="6.44" y2="6.5775" width="0.2032" layer="1"/>
+<wire x1="5.715" y1="6.5775" x2="6.44" y2="6.5775" width="0.2032" layer="1"/>
+<contactref element="D1" pad="C"/>
+<wire x1="7.3025" y1="6.7025" x2="7.3025" y2="6.6675" width="0.2032" layer="1"/>
+<wire x1="7.3025" y1="6.6675" x2="6.82625" y2="6.19125" width="0.2032" layer="1"/>
+<wire x1="10.94" y1="1.27" x2="8.89" y2="2.71" width="0" layer="19" extent="1-1"/>
 </signal>
 <signal name="VIN">
@@
 <contactref element="JP1" pad="1"/>
 <contactref element="JP3" pad="1"/>
-<contactref element="Q3" pad="2"/>
-<contactref element="R4" pad="2"/>
 <contactref element="R6" pad="1"/>
 <polygon width="0.2032" layer="1" isolate="0.5" thermals="no">
@@
 <via x="6.35" y="3.175" extent="1-16" drill="0.4" diameter="0.3"/>
 <via x="1.27" y="6.35" extent="1-16" drill="0.4" diameter="0.3"/>
-<contactref element="Q4" pad="2"/>
-<wire x1="1.27" y1="1.27" x2="11.16" y2="-1.59" width="0" layer="19" extent="1-1"/>
+<contactref element="R4" pad="1"/>
+<wire x1="6.35" y1="13.97" x2="8.89" y2="13.97" width="0" layer="19" extent="1-1"/>
+<wire x1="10.16" y1="10.795" x2="8.89" y2="13.97" width="0" layer="19" extent="1-1"/>
+<wire x1="11.7475" y1="9.7525" x2="10.16" y2="10.795" width="0" layer="19" extent="1-1"/>
+<wire x1="11.2825" y1="5.7175" x2="11.7475" y2="9.7525" width="0" layer="19" extent="1-1"/>
+<wire x1="9.525" y1="5.08" x2="11.2825" y2="5.7175" width="0" layer="19" extent="1-1"/>
+<wire x1="9.2075" y1="6.3025" x2="9.525" y2="5.08" width="0" layer="19" extent="1-1"/>
+<wire x1="13.335" y1="5.08" x2="11.2825" y2="5.7175" width="0" layer="19" extent="1-1"/>
+<wire x1="6.715" y1="4.1275" x2="9.525" y2="5.08" width="0" layer="19" extent="1-1"/>
+<wire x1="6.35" y1="5.08" x2="6.715" y2="4.1275" width="0" layer="19" extent="1-1"/>
+<wire x1="6.35" y1="3.175" x2="6.715" y2="4.1275" width="0" layer="19" extent="1-1"/>
+<wire x1="1.27" y1="13.97" x2="6.35" y2="13.97" width="0" layer="19" extent="1-1"/>
+<wire x1="1.27" y1="6.35" x2="6.35" y2="5.08" width="0" layer="19" extent="1-1"/>
+<wire x1="1.27" y1="1.27" x2="1.27" y2="6.35" width="0" layer="19" extent="1-1"/>
+<wire x1="-0.725" y1="-6.35" x2="1.27" y2="1.27" width="0" layer="19" extent="1-1"/>
 </signal>
 <signal name="N$4">
@@
 <wire x1="7.3025" y1="8.0025" x2="7.595" y2="8.0025" width="0.2032" layer="1"/>
 <wire x1="7.595" y1="8.0025" x2="7.62" y2="8.0275" width="0.2032" layer="1"/>
+<contactref element="R4" pad="2"/>
+<wire x1="0.725" y1="-6.35" x2="5.715" y2="8.0275" width="0" layer="19" extent="1-1"/>
 </signal>
 <signal name="N$3">
@@
 <wire x1="11.7475" y1="13.4747" x2="11.43" y2="13.97" width="0.2032" layer="1"/>
 </signal>
-<signal name="N$45">
-<contactref element="Q3" pad="3"/>
-<contactref element="R3" pad="2"/>
-<contactref element="R2" pad="1"/>
-<wire x1="4.1275" y1="6.5775" x2="5.715" y2="6.5775" width="0.2032" layer="1"/>
-<wire x1="8.89" y1="4.1275" x2="8.89" y2="2.71" width="0.2032" layer="1"/>
-<wire x1="8.89" y1="2.71" x2="9.06" y2="2.54" width="0.2032" layer="1"/>
-<wire x1="8.89" y1="4.1275" x2="6.82625" y2="6.19125" width="0.2032" layer="1"/>
-<wire x1="6.82625" y1="6.19125" x2="6.44" y2="6.5775" width="0.2032" layer="1"/>
-<wire x1="5.715" y1="6.5775" x2="6.44" y2="6.5775" width="0.2032" layer="1"/>
-<contactref element="D1" pad="C"/>
-<wire x1="7.3025" y1="6.7025" x2="7.3025" y2="6.6675" width="0.2032" layer="1"/>
-<wire x1="7.3025" y1="6.6675" x2="6.82625" y2="6.19125" width="0.2032" layer="1"/>
-</signal>
 </signals>

Commit message: Toggle updated
Parts:
- Q1: value (none) -> PFET
- Q2: value MOSFET-NCHANNELBSS123LT1G -> NFET
- R5, R6: value 10k -> 100R
Changed lines of the file:
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@@
 <attribute name="NAME" x="2.794" y="5.6515" size="1.016" layer="25" ratio="15" rot="R90"/>
 </element>
-<element name="Q1" library="transistor-power" package="MICRO3" value="" x="3.4925" y="10.795" smashed="yes" rot="R90">
+<element name="Q1" library="transistor-power" package="MICRO3" value="PFET" x="3.4925" y="10.795" smashed="yes" rot="R90">
 <attribute name="NAME" x="1.575" y="10.30625" size="0.762" layer="25" ratio="15" rot="R90"/>
 <attribute name="VALUE" x="6.8925" y="9.295" size="1.778" layer="27" rot="R90"/>
@@
 <attribute name="NAME" x="5.08" y="5.08" size="0.762" layer="25" font="vector" ratio="15"/>
 </element>
-<element name="Q2" library="SparkFun-DiscreteSemi" package="SOT23" value="MOSFET-NCHANNELBSS123LT1G" x="12.3825" y="6.6675" smashed="yes" rot="R270">
+<element name="Q2" library="SparkFun-DiscreteSemi" package="SOT23" value="NFET" x="12.3825" y="6.6675" smashed="yes" rot="R270">
 <attribute name="PROD_ID" value="TRANS-08345" x="12.3825" y="6.6675" size="1.778" layer="27" rot="R270" display="off"/>
 <attribute name="NAME" x="13.3985" y="7.747" size="0.762" layer="25" ratio="15"/>
@@
 </element>
 <element name="BUT" library="SparkFun-Connectors" package="1X02_NO_SILK" value="M021X02_NO_SILK" x="11.43" y="13.97" smashed="yes"/>
-<element name="R5" library="wes" package="R0603" value="10k" x="13.6525" y="10.4775" smashed="yes" rot="R90">
+<element name="R5" library="wes" package="R0603" value="100R" x="13.6525" y="10.4775" smashed="yes" rot="R90">
 <attribute name="NAME" x="13.0175" y="11.90625" size="0.762" layer="25" font="vector" ratio="15"/>
 </element>
-<element name="R6" library="wes" package="R0603" value="10k" x="11.7475" y="10.4775" smashed="yes" rot="R90">
+<element name="R6" library="wes" package="R0603" value="100R" x="11.7475" y="10.4775" smashed="yes" rot="R90">
 <attribute name="NAME" x="11.1125" y="11.90625" size="0.762" layer="25" font="vector" ratio="15"/>
 </element>
