File: Eletrônica/Toggle/Toggle.sch (EAGLE design)
At the start: 17 parts, among them Q1 IRLML5203, Q2 MOSFET-NCHANNELBSS123LT1G, Q3 MOSFET-NCHANNELBSS123LT1G, Q4 IRLML5203

Commit message: Eagle .gitignore updates
Parts:
- removed Q3: MOSFET-NCHANNELBSS123LT1G, SparkFun-DiscreteSemi:MOSFET-NCHANNELBSS123LT1G
- removed Q4: IRLML5203, transistor-power:IRLML5203
- R2, R4: value 100k -> 1M
Connections:
- removed net N$45: D1.C, Q3.D, R2.1, R3.2
- net ARD_OFF: now also D1.C, R2.1, R3.2; no longer Q3.G, Q4.G, R4.1
- net GND: now also R4.1; no longer Q3.S, Q4.S, R4.2
- net N$2: now also R4.2
Changed lines of the file:
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@@
 <part name="R1" library="wes" deviceset="R-EU_" device="R0603" value="10k"/>
 <part name="Q1" library="transistor-power" deviceset="IRLML5203" device="" value=""/>
-<part name="R2" library="wes" deviceset="R-EU_" device="R0603" value="100k"/>
+<part name="R2" library="wes" deviceset="R-EU_" device="R0603" value="1M"/>
 <part name="SUPPLY1" library="SparkFun-Aesthetics" deviceset="VIN" device=""/>
 <part name="VOUT" library="supply1" deviceset="VCC" device=""/>
@@
 <part name="JP3" library="SparkFun-Connectors" deviceset="M03" device="1X03_NO_SILK"/>
 <part name="BUT" library="SparkFun-Connectors" deviceset="M02" device="1X02_NO_SILK" value="M021X02_NO_SILK"/>
-<part name="Q3" library="SparkFun-DiscreteSemi" deviceset="MOSFET-NCHANNEL" device="BSS123LT1G" value="MOSFET-NCHANNELBSS123LT1G"/>
-<part name="R4" library="wes" deviceset="R-EU_" device="R0603" value="100k"/>
 <part name="R5" library="wes" deviceset="R-EU_" device="R0603" value="10k"/>
 <part name="R6" library="wes" deviceset="R-EU_" device="R0603" value="10k"/>
 <part name="D1" library="SparkFun-DiscreteSemi" deviceset="DIODE" device="SOD523"/>
-<part name="Q4" library="transistor-power" deviceset="IRLML5203" device="" value=""/>
+<part name="R4" library="wes" deviceset="R-EU_" device="R0603" value="1M"/>
 </parts>
 <sheets>
@@
 DigitalWrite(6, LOW);</text>
 <text x="40.64" y="66.04" size="1.778" layer="97">From Battery</text>
-<wire x1="187.96" y1="-2.54" x2="187.96" y2="86.36" width="0.1524" layer="94" style="longdash"/>
 <text x="7.62" y="78.74" size="2.54" layer="94">Power Toggle</text>
 </plain>
@@
 <instance part="JP3" gate="G$1" x="162.56" y="58.42" rot="R180"/>
 <instance part="BUT" gate="G$1" x="25.4" y="38.1"/>
-<instance part="Q3" gate="G$1" x="88.9" y="15.24" rot="MR0"/>
-<instance part="R4" gate="G$1" x="101.6" y="7.62" smashed="yes" rot="R270"/>
 <instance part="R5" gate="G$1" x="40.64" y="40.64" smashed="yes" rot="R180">
 <attribute name="NAME" x="39.5986" y="36.83" size="1.778" layer="95" rot="R270"/>
@@
 </instance>
 <instance part="D1" gate="G$1" x="81.28" y="25.4"/>
-<instance part="Q4" gate="G$1" x="91.44" y="-15.24" smashed="yes" rot="R180">
-<attribute name="NAME" x="78.74" y="-17.78" size="1.778" layer="95" rot="R90"/>
-<attribute name="VALUE" x="81.28" y="-17.78" size="1.778" layer="96" rot="R90"/>
+<instance part="R4" gate="G$1" x="68.58" y="12.7" smashed="yes" rot="R90">
+<attribute name="NAME" x="57.15" y="14.1986" size="1.778" layer="95"/>
+<attribute name="VALUE" x="57.15" y="11.938" size="1.778" layer="96"/>
 </instance>
 </instances>
@@
 </segment>
 <segment>
-<pinref part="Q3" gate="G$1" pin="G"/>
-<wire x1="96.52" y1="15.24" x2="101.6" y2="15.24" width="0.1524" layer="91"/>
-<pinref part="R4" gate="G$1" pin="1"/>
-<wire x1="101.6" y1="15.24" x2="101.6" y2="12.7" width="0.1524" layer="91"/>
-<wire x1="101.6" y1="15.24" x2="106.68" y2="15.24" width="0.1524" layer="91"/>
-<pinref part="Q4" gate="G$1" pin="G"/>
-<wire x1="93.98" y1="-17.78" x2="106.68" y2="-17.78" width="0.1524" layer="91"/>
-<wire x1="106.68" y1="-17.78" x2="106.68" y2="15.24" width="0.1524" layer="91"/>
+<pinref part="R2" gate="G$1" pin="1"/>
+<wire x1="88.9" y1="30.48" x2="88.9" y2="40.64" width="0.1524" layer="91"/>
+<label x="139.7" y="10.16" size="1.778" layer="95"/>
+<pinref part="R3" gate="G$1" pin="2"/>
+<wire x1="86.36" y1="30.48" x2="88.9" y2="30.48" width="0.1524" layer="91"/>
+<pinref part="D1" gate="G$1" pin="C"/>
+<wire x1="83.82" y1="25.4" x2="86.36" y2="25.4" width="0.1524" layer="91"/>
+<wire x1="86.36" y1="25.4" x2="86.36" y2="30.48" width="0.1524" layer="91"/>
+<wire x1="88.9" y1="30.48" x2="96.52" y2="30.48" width="0.1524" layer="91"/>
+<label x="96.52" y="30.48" size="1.778" layer="95"/>
 </segment>
 </net>
@@
 <pinref part="C2" gate="G$1" pin="2"/>
 <wire x1="63.5" y1="-2.54" x2="63.5" y2="-5.08" width="0.1524" layer="91"/>
-<wire x1="73.66" y1="7.62" x2="73.66" y2="-2.54" width="0.1524" layer="91"/>
+<wire x1="73.66" y1="7.62" x2="73.66" y2="5.08" width="0.1524" layer="91"/>
+<wire x1="73.66" y1="5.08" x2="73.66" y2="-2.54" width="0.1524" layer="91"/>
 <wire x1="73.66" y1="-2.54" x2="63.5" y2="-2.54" width="0.1524" layer="91"/>
 <pinref part="Q2" gate="G$1" pin="S"/>
 <junction x="63.5" y="-2.54"/>
-<wire x1="73.66" y1="-2.54" x2="81.28" y2="-2.54" width="0.1524" layer="91"/>
-<pinref part="Q3" gate="G$1" pin="S"/>
-<wire x1="81.28" y1="-2.54" x2="88.9" y2="-2.54" width="0.1524" layer="91"/>
-<wire x1="88.9" y1="-2.54" x2="88.9" y2="10.16" width="0.1524" layer="91"/>
-<pinref part="R4" gate="G$1" pin="2"/>
-<wire x1="101.6" y1="2.54" x2="101.6" y2="-2.54" width="0.1524" layer="91"/>
-<wire x1="101.6" y1="-2.54" x2="88.9" y2="-2.54" width="0.1524" layer="91"/>
-<junction x="73.66" y="-2.54"/>
-<junction x="88.9" y="-2.54"/>
 <pinref part="R6" gate="G$1" pin="1"/>
 <wire x1="45.72" y1="38.1" x2="50.8" y2="38.1" width="0.1524" layer="91"/>
 <wire x1="50.8" y1="38.1" x2="50.8" y2="-2.54" width="0.1524" layer="91"/>
 <wire x1="50.8" y1="-2.54" x2="63.5" y2="-2.54" width="0.1524" layer="91"/>
-<pinref part="Q4" gate="G$1" pin="S"/>
-<wire x1="88.9" y1="-20.32" x2="81.28" y2="-20.32" width="0.1524" layer="91"/>
-<wire x1="81.28" y1="-20.32" x2="81.28" y2="-2.54" width="0.1524" layer="91"/>
+<pinref part="R4" gate="G$1" pin="1"/>
+<wire x1="68.58" y1="7.62" x2="68.58" y2="5.08" width="0.1524" layer="91"/>
+<wire x1="68.58" y1="5.08" x2="73.66" y2="5.08" width="0.1524" layer="91"/>
 </segment>
 <segment>
@@
 <wire x1="71.12" y1="30.48" x2="73.66" y2="30.48" width="0.1524" layer="91"/>
 <pinref part="C2" gate="G$1" pin="1"/>
-<wire x1="73.66" y1="15.24" x2="73.66" y2="30.48" width="0.1524" layer="91"/>
+<wire x1="73.66" y1="15.24" x2="73.66" y2="20.32" width="0.1524" layer="91"/>
 <pinref part="R3" gate="G$1" pin="1"/>
+<wire x1="73.66" y1="20.32" x2="73.66" y2="30.48" width="0.1524" layer="91"/>
 <wire x1="76.2" y1="30.48" x2="73.66" y2="30.48" width="0.1524" layer="91"/>
 <pinref part="Q2" gate="G$1" pin="G"/>
@@
 <wire x1="78.74" y1="25.4" x2="76.2" y2="25.4" width="0.1524" layer="91"/>
 <wire x1="76.2" y1="25.4" x2="76.2" y2="30.48" width="0.1524" layer="91"/>
+<pinref part="R4" gate="G$1" pin="2"/>
+<wire x1="68.58" y1="17.78" x2="68.58" y2="20.32" width="0.1524" layer="91"/>
+<wire x1="68.58" y1="20.32" x2="73.66" y2="20.32" width="0.1524" layer="91"/>
 </segment>
 </net>
@@
 </segment>
 </net>
-<net name="N$45" class="0">
-<segment>
-<pinref part="R2" gate="G$1" pin="1"/>
-<wire x1="88.9" y1="30.48" x2="88.9" y2="40.64" width="0.1524" layer="91"/>
-<label x="139.7" y="10.16" size="1.778" layer="95"/>
-<pinref part="R3" gate="G$1" pin="2"/>
-<wire x1="86.36" y1="30.48" x2="88.9" y2="30.48" width="0.1524" layer="91"/>
-<junction x="88.9" y="30.48"/>
-<pinref part="Q3" gate="G$1" pin="D"/>
-<wire x1="88.9" y1="30.48" x2="88.9" y2="20.32" width="0.1524" layer="91"/>
-<pinref part="D1" gate="G$1" pin="C"/>
-<wire x1="83.82" y1="25.4" x2="86.36" y2="25.4" width="0.1524" layer="91"/>
-<wire x1="86.36" y1="25.4" x2="86.36" y2="30.48" width="0.1524" layer="91"/>
-</segment>
-</net>

Commit message: Toggle updated
Parts:
- Q1: value IRLML5203 -> PFET
- Q2: value MOSFET-NCHANNELBSS123LT1G -> NFET
- R5, R6: value 10k -> 100R
Changed lines of the file:
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@@
 <parts>
 <part name="R1" library="wes" deviceset="R-EU_" device="R0603" value="10k"/>
-<part name="Q1" library="transistor-power" deviceset="IRLML5203" device="" value=""/>
+<part name="Q1" library="transistor-power" deviceset="IRLML5203" device="" value="PFET"/>
 <part name="R2" library="wes" deviceset="R-EU_" device="R0603" value="1M"/>
 <part name="SUPPLY1" library="SparkFun-Aesthetics" deviceset="VIN" device=""/>
@@
 <part name="C2" library="wes" deviceset="C-EU" device="C0805" value="10uF 10V"/>
 <part name="R3" library="wes" deviceset="R-EU_" device="R0603" value="0R"/>
-<part name="Q2" library="SparkFun-DiscreteSemi" deviceset="MOSFET-NCHANNEL" device="BSS123LT1G" value="MOSFET-NCHANNELBSS123LT1G"/>
+<part name="Q2" library="SparkFun-DiscreteSemi" deviceset="MOSFET-NCHANNEL" device="BSS123LT1G" value="NFET"/>
 <part name="JP1" library="SparkFun-Connectors" deviceset="M02" device="1X02_NO_SILK" value="M021X02_NO_SILK"/>
 <part name="JP3" library="SparkFun-Connectors" deviceset="M03" device="1X03_NO_SILK"/>
 <part name="BUT" library="SparkFun-Connectors" deviceset="M02" device="1X02_NO_SILK" value="M021X02_NO_SILK"/>
-<part name="R5" library="wes" deviceset="R-EU_" device="R0603" value="10k"/>
-<part name="R6" library="wes" deviceset="R-EU_" device="R0603" value="10k"/>
+<part name="R5" library="wes" deviceset="R-EU_" device="R0603" value="100R"/>
+<part name="R6" library="wes" deviceset="R-EU_" device="R0603" value="100R"/>
 <part name="D1" library="SparkFun-DiscreteSemi" deviceset="DIODE" device="SOD523"/>
 <part name="R4" library="wes" deviceset="R-EU_" device="R0603" value="1M"/>
@@
 <instance part="BUT" gate="G$1" x="25.4" y="38.1"/>
 <instance part="R5" gate="G$1" x="40.64" y="40.64" smashed="yes" rot="R180">
-<attribute name="NAME" x="39.5986" y="36.83" size="1.778" layer="95" rot="R270"/>
-<attribute name="VALUE" x="42.418" y="36.83" size="1.778" layer="96" rot="R270"/>
+<attribute name="NAME" x="34.29" y="44.6786" size="1.778" layer="95"/>
+<attribute name="VALUE" x="39.37" y="44.958" size="1.778" layer="96"/>
 </instance>
 <instance part="R6" gate="G$1" x="40.64" y="38.1" smashed="yes" rot="R180">
-<attribute name="NAME" x="39.5986" y="34.29" size="1.778" layer="95" rot="R270"/>
-<attribute name="VALUE" x="42.418" y="34.29" size="1.778" layer="96" rot="R270"/>
+<attribute name="NAME" x="34.29" y="42.1386" size="1.778" layer="95"/>
+<attribute name="VALUE" x="39.37" y="42.418" size="1.778" layer="96"/>
 </instance>
 <instance part="D1" gate="G$1" x="81.28" y="25.4"/>
