File: Eletrônica/Principal/Pluvion 1 - Rev A.brd (EAGLE design)
At the start: 160 x 100 mm, 27 parts, among them IC1 REG1117, J1 22-05-7048-04, Q1 PFET, Q2 NFET

Commit message: Eagle Rev A
Parts:
- removed C3: (no value), wes:C0805
- removed J1: 22-05-7048-04, con-molex:7395-04
- removed MDL1: (no value), ESP8266-ESP12E:ESP8266-ESP12E
- added D6: DB2S31600, SparkFun-DiscreteSemi:SMA-DIODE
- added J3, J4: 22-05-7048-04, con-molex:7395-04
- added J5: 22-05-7028-02, con-molex:7395-02
- added JP2, JP3: JUMPER-3-OLDSMD, SparkFun-Passives:SJ_3
- added JP4: FTDI_BASICPTH, SparkFun-Connectors:FTDI_BASIC
- added JP5: (no value), SparkFun-Passives:1X02
- added JP6: (no value), SparkFun-Passives:SJ_2S-NO
- added LED1: (no value), SparkFun-LED:LED-1206
- added MDL2: (no value), ESP8266-ESP12E:ESP8266-ESP12E
- added Q3, Q4: S8050, semicon-smd-ipc:SOT23
- added R10, R11, R18, R8, R9: (no value), wes:R0805
- added RN2: (no value), resistor-dil:0603-ARV
- added RN3: 10K, resistor-dil:0603-ARV
- added RN6: 1K, resistor-dil:0603-ARV
- added SW1: Reset, buttons:BT4.5X4.5
- C1, C2: device wes:PANASONIC_D -> wes:PANASONIC_C
- JP1: value M021X02_NO_SILK -> USB_MICROB_PLUGCONN-11752; device SparkFun-Connectors:1X02_NO_SILK -> SparkFun-Connectors:USB-B-MICRO-SMD_V03
- moved R6 54.8 mm to (21.6, 12.7), flipped to the bottom, turned to 90 degrees
- moved C5 45.7 mm to (17.8, 34.9)
- moved U1 28.2 mm to (41.9, 36.8)
- moved R5 25.1 mm to (6.35, 11.4), turned to 270 degrees
- moved Q2 23.9 mm to (5.08, 16.5), turned to 180 degrees
- moved JP1 20.7 mm to (14.0, 3.81), turned to 90 degrees
- moved R4 20.7 mm to (3.81, 21.6), turned to 270 degrees
- moved C1 20.3 mm to (6.99, 27.9), turned to 90 degrees
- moved C6 19.3 mm to (11.4, 27.9), turned to 270 degrees
- moved C7 19.3 mm to (6.35, 21.6), turned to 90 degrees
- moved R1 18.5 mm to (8.89, 11.4), turned to 270 degrees
- moved U$1 16.1 mm to (23.7, 6.73), flipped to the bottom, turned to 90 degrees
- moved D2 14.6 mm to (17.1, 46.4), flipped to the bottom
- moved D3 14.6 mm to (17.1, 43.8), flipped to the bottom, turned to 180 degrees
- moved R7 14.6 mm to (17.1, 48.9), flipped to the bottom, turned to 180 degrees
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Connections:
- removed net 3.3V: C2.+, C4.1, C5.1, D2.1, IC1.2, R7.2, U1.VDD
- removed net N$5: D2.2, D3.1, R6.2, R7.1
- removed net VOUT: C6.1, D5.C
- new net +3V3: C2.+, C4.1, C5.1, D2.1, D6.C, IC1.2, JP2.1, JP3.1, MDL2.8, R7.2, R8.1, R9.1, RN3.1, RN3.6, RN3.7, U1.VDD
- new net +5V: C1.+, C6.1, D5.C, IC1.3, JP2.3, JP3.3, JP5.2, JP6.2
- new net CH_PD: MDL2.3, R8.2
- new net D1: RN3.8, RN6.6, U1.DATA
- new net D2: RN6.5
- new net D5: D2.2, D3.1, MDL2.5, R6.2, R7.1
- new net DTR: JP4.DTR, Q4.2, R10.2
- new net GPIO0: MDL2.12, Q4.3, RN3.2
- new net GPIO15: MDL2.10, RN3.4
- new net GPIO2: MDL2.11, RN3.3
- new net N$10: MDL2.7
- new net N$11: MDL2.4
- new net N$12: MDL2.6
- new net N$14: MDL2.2
- new net N$16: RN2.7
- new net N$17: J4.3, RN2.3
- new net N$18: J3.2, JP2.2
- new net N$19: J4.4, RN2.4
- new net N$20: J4.2, JP3.2
- new net N$21: RN2.6
- new net N$22: RN2.5
- new net N$25: MDL2.14, RN6.3
- new net N$27: D6.A, JP4.VCC
- new net N$30: MDL2.13, RN6.4
- new net N$33: LED1.A, R18.1
- new net N$34: JP6.1, R18.2
- new net N$6: Q3.1, R10.1
- new net N$7: Q4.1, R11.1
- new net N$9: RN2.8
- new net RST: MDL2.1, Q3.2, R9.2, SW1.P, SW1.P1
- new net RTS: JP4.CTS, Q3.3, R11.2
- new net RX: MDL2.16, RN6.1
- new net TX: MDL2.15, RN6.2
- new net _RX: JP4.RXI, RN6.8
- new net _TX: JP4.TXO, RN6.7
- net GND: now also J3.1, J4.1, J5.1, JP1.GND1, JP4.GND, LED1.C, MDL2.9, RN3.5, SW1.S, SW1.S1; no longer C3.2, JP1.1
- net N$3: now also J3.3, RN2.1; no longer C1.+, C3.1, IC1.3
- net N$4: now also J3.4, RN2.2; no longer U1.DATA
- net VIN: now also J5.2, JP1.VBUS1, JP5.1; no longer JP1.2
Routing:
- net +3V3: track 0.00 -> 159.7 mm, vias 0 -> 3
- net +5V: track 0.00 -> 108.5 mm
- net RST: track 0.00 -> 58.9 mm, vias 0 -> 4
- net D5: track 0.00 -> 54.9 mm, vias 0 -> 5
- net _RX: track 0.00 -> 52.7 mm
- net _TX: track 0.00 -> 48.7 mm
- net HALL: track 0.00 -> 36.0 mm, vias 0 -> 1
- net VIN: track 0.00 -> 35.8 mm
- net GPIO0: track 0.00 -> 33.9 mm, vias 0 -> 2
- net D1: track 0.00 -> 22.6 mm
- net RTS: track 0.00 -> 13.0 mm
- net DTR: track 0.00 -> 12.1 mm
- net N$19: track 0.00 -> 11.3 mm
- net N$2: track 0.00 -> 11.0 mm
- net N$17: track 0.00 -> 9.79 mm
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- added copper zone on layer 16, net GND
Other:
- board size 160 x 100 mm -> 50 x 65 mm

Commit message: Prototype BOM
Parts:
- C4, C5: value (none) -> 100nF
- R10, R11, RN2: value (none) -> 1k
- R18, R7, R8, R9: value (none) -> 10k
- R3: value 0R -> 100R
- R6: value (none) -> 100R
Changed lines of the file:
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@@
 <attribute name="OC_FARNELL" value="1097566" x="16.51" y="29.21" size="1.778" layer="27" rot="R180" display="off"/>
 </element>
-<element name="C4" library="wes" package="C0805" value="" x="22.86" y="18.415" rot="R180"/>
+<element name="C4" library="wes" package="C0805" value="100nF" x="22.86" y="18.415" rot="R180"/>
 <element name="U1" library="RHT03_DHT-22_AM2302" package="RHT03_DHT-22/RA" value="" x="41.91" y="36.83">
 <attribute name="PROD_ID" value="SEN-10167" x="41.91" y="36.83" size="1.778" layer="27" display="off"/>
 </element>
-<element name="C5" library="wes" package="C0805" value="" x="17.78" y="34.925"/>
+<element name="C5" library="wes" package="C0805" value="100nF" x="17.78" y="34.925"/>
 <element name="C6" library="wes" package="C0805" value="10uF 10V" x="11.43" y="27.94" smashed="yes" rot="R270">
 <attribute name="NAME" x="10.795" y="25.24125" size="0.762" layer="25" ratio="15"/>
@@
 <attribute name="NAME" x="14.605" y="23.8125" size="0.762" layer="25" font="vector" ratio="15" rot="R180"/>
 </element>
-<element name="R3" library="wes" package="R0805" value="0R" x="8.89" y="21.59" smashed="yes" rot="R90">
+<element name="R3" library="wes" package="R0805" value="100R" x="8.89" y="21.59" smashed="yes" rot="R90">
 <attribute name="NAME" x="9.525" y="23.8125" size="0.762" layer="25" font="vector" ratio="15" rot="R180"/>
 </element>
@@
 <element name="R4" library="wes" package="R0805" value="1M" x="3.81" y="21.59" rot="R270"/>
 <element name="U$1" library="lib_pluvion" package="SOT23" value="DRV5023FAQDBZR" x="23.73" y="6.73" rot="MR90"/>
-<element name="R6" library="wes" package="R0805" value="" x="21.59" y="12.7" rot="MR90"/>
-<element name="R7" library="wes" package="R0805" value="" x="17.145" y="48.895" rot="MR180"/>
+<element name="R6" library="wes" package="R0805" value="100R" x="21.59" y="12.7" rot="MR90"/>
+<element name="R7" library="wes" package="R0805" value="10k" x="17.145" y="48.895" rot="MR180"/>
 <element name="D2" library="SparkFun-DiscreteSemi" package="SOD-323" value="" x="17.145" y="46.355" rot="MR0">
 <attribute name="PROD_ID" value="DIO-09646" x="17.145" y="46.355" size="1.778" layer="28" rot="MR0" display="off"/>
@@
 <element name="Q3" library="semicon-smd-ipc" package="SOT23" value="S8050" x="30.48" y="31.75" rot="R90"/>
 <element name="Q4" library="semicon-smd-ipc" package="SOT23" value="S8050" x="27.305" y="22.225" rot="R90"/>
-<element name="R8" library="wes" package="R0805" value="" x="4.445" y="52.705"/>
-<element name="R9" library="wes" package="R0805" value="" x="4.445" y="56.515"/>
+<element name="R8" library="wes" package="R0805" value="10k" x="4.445" y="52.705"/>
+<element name="R9" library="wes" package="R0805" value="10k" x="4.445" y="56.515"/>
 <element name="MDL2" library="ESP8266-ESP12E" package="ESP8266-ESP12E" value="" x="16.51" y="50.8"/>
 <element name="JP2" library="SparkFun-Passives" package="SJ_3" value="JUMPER-3-OLDSMD" x="40.64" y="16.51"/>
@@
 <attribute name="OC_FARNELL" value="unknown" x="26.67" y="30.48" size="1.778" layer="27" display="off"/>
 </element>
-<element name="RN2" library="resistor-dil" package="0603-ARV" value="" x="33.655" y="17.78" rot="MR0">
+<element name="RN2" library="resistor-dil" package="0603-ARV" value="1k" x="33.655" y="17.78" rot="MR0">
 <attribute name="MF" value="" x="56.515" y="50.8" size="1.778" layer="28" rot="MR0" display="off"/>
 <attribute name="MPN" value="" x="56.515" y="50.8" size="1.778" layer="28" rot="MR0" display="off"/>
@@
 </element>
 <element name="LED1" library="SparkFun-LED" package="LED-1206" value="" x="46.99" y="5.08" rot="R270"/>
-<element name="R18" library="wes" package="R0805" value="" x="46.99" y="10.16" rot="R90"/>
+<element name="R18" library="wes" package="R0805" value="10k" x="46.99" y="10.16" rot="R90"/>
 <element name="JP6" library="SparkFun-Passives" package="SJ_2S-NO" value="" x="46.99" y="13.97" rot="R90"/>
 <element name="RN3" library="resistor-dil" package="0603-ARV" value="10K" x="30.48" y="46.99" rot="R270">
@@
 </element>
 <element name="D6" library="SparkFun-DiscreteSemi" package="SMA-DIODE" value="DB2S31600" x="33.02" y="26.035" rot="R90"/>
-<element name="R10" library="wes" package="R0805" value="" x="29.5275" y="26.67" rot="R270"/>
-<element name="R11" library="wes" package="R0805" value="" x="27.305" y="26.67" rot="R90"/>
+<element name="R10" library="wes" package="R0805" value="1k" x="29.5275" y="26.67" rot="R270"/>
+<element name="R11" library="wes" package="R0805" value="1k" x="27.305" y="26.67" rot="R90"/>
 </elements>
 <signals>
