File: Eletrônica/Principal/Pluvion 1 - Rev A.brd (EAGLE design)
At the start: 50 x 65 mm, 46 parts, among them IC1 REG1117, J3 22-05-7048-04, J4 22-05-7048-04, J5 22-05-7028-02, Q1 PFET, Q2 NFET, Q3 S8050, Q4 S8050, SW1 Reset

Commit message: Pluvion 1 Rev C
Connections:
- net RST: now also Q3.3; no longer Q3.2
- net RTS: now also Q3.2; no longer Q3.3
Routing:
- net RTS: track 13.0 -> 9.23 mm
Changed lines of the file:
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@@
 <?xml version="1.0" encoding="utf-8"?>
 <!DOCTYPE eagle SYSTEM "eagle.dtd">
-<eagle version="7.6.0">
+<eagle version="7.3.0">
 <drawing>
 <settings>
@@
 </signal>
 <signal name="RST">
-<contactref element="Q3" pad="2"/>
 <contactref element="R9" pad="2"/>
 <via x="24.765" y="34.925" extent="1-16" drill="0.8" diameter="1.6"/>
@@
 <wire x1="31.115" y1="35.56" x2="31.75" y2="34.925" width="0.4064" layer="1"/>
 <wire x1="31.75" y1="34.925" x2="31.75" y2="32.87" width="0.4064" layer="1"/>
-<wire x1="31.75" y1="32.87" x2="31.58" y2="32.7" width="0.4064" layer="1"/>
 <contactref element="SW1" pad="P"/>
 <contactref element="SW1" pad="P1"/>
@@
 <wire x1="31.115" y1="35.56" x2="25.4" y2="35.56" width="0.4064" layer="1"/>
 <wire x1="25.4" y1="35.56" x2="24.765" y2="34.925" width="0.4064" layer="1"/>
+<contactref element="Q3" pad="3"/>
+<wire x1="31.75" y1="32.87" x2="29.38" y2="31.75" width="0" layer="19" extent="1-1"/>
 </signal>
 <signal name="D5">
@@
 </signal>
 <signal name="RTS">
-<contactref element="Q3" pad="3"/>
 <contactref element="JP4" pad="CTS"/>
 <contactref element="R11" pad="2"/>
 <wire x1="27.305" y1="27.545" x2="27.305" y2="29.845" width="0.4064" layer="1"/>
 <wire x1="27.305" y1="29.845" x2="29.21" y2="31.75" width="0.4064" layer="1"/>
-<wire x1="29.21" y1="31.75" x2="29.38" y2="31.75" width="0.4064" layer="1"/>
-<wire x1="29.38" y1="31.75" x2="33.02" y2="31.75" width="0.4064" layer="1"/>
 <wire x1="33.02" y1="31.75" x2="34.29" y2="30.48" width="0.4064" layer="1"/>
 <wire x1="34.29" y1="30.48" x2="36.73" y2="30.48" width="0.4064" layer="1"/>
+<contactref element="Q3" pad="2"/>
+<wire x1="31.58" y1="32.7" x2="33.02" y2="31.75" width="0" layer="19" extent="1-1"/>
+<wire x1="29.21" y1="31.75" x2="31.58" y2="32.7" width="0" layer="19" extent="1-1"/>
 </signal>
 <signal name="DTR">
