File: Eletrônica/Principal/Pluvion 1 - Rev A.sch (EAGLE design)
At the start: 27 parts, among them IC1 REG1117, J1 22-05-7048-04, Q1 PFET, Q2 NFET

Commit message: Eagle Rev A
Parts:
- removed C3: (no value), wes:C-EUC0805
- removed J1: 22-05-7048-04, con-molex:22-05-7048-04
- removed MDL1: (no value), ESP8266-ESP12E:ESP8266-12EESP8266-ESP12E
- added D6: DB2S31600, SparkFun-DiscreteSemi:DIODESMA
- added J3, J4: 22-05-7048-04, con-molex:22-05-7048-04
- added J5: 22-05-7028-02, con-molex:22-05-7028-02
- added JP2, JP3: JUMPER-3-OLDSMD, SparkFun-Passives:JUMPER-3-OLDSMD
- added JP4: FTDI_BASICPTH, SparkFun-Connectors:FTDI_BASICPTH
- added JP5: (no value), SparkFun-Passives:JUMPER-2PTH
- added JP6: (no value), SparkFun-Passives:JUMPER-2SMD-NO
- added LED1: (no value), SparkFun-LED:LED1206
- added MDL2: (no value), ESP8266-ESP12E:ESP8266-12EESP8266-ESP12E
- added Q3, Q4: S8050, semicon-smd-ipc:NPN-TRANSISTOR_SOT23
- added R10, R11, R18, R8, R9: (no value), wes:R-EU_R0805
- added RN2: (no value), resistor-dil:4R-N0603-ARV
- added RN3: 10K, resistor-dil:4R-N0603-ARV
- added RN6: 1K, resistor-dil:4R-N0603-ARV
- added SW1: Reset, buttons:10-XX-4.5SMD
- C1, C2: device wes:CPOL-EUD -> wes:CPOL-EUC
- JP1: value M021X02_NO_SILK -> USB_MICROB_PLUGCONN-11752; device SparkFun-Connectors:M021X02_NO_SILK -> SparkFun-Connectors:USB_MICROB_PLUGCONN-11752
Connections:
- removed net 3.3V: C2.+, C4.1, C5.1, D2.C, IC1.VOUT, R7.2, U1.VDD
- removed net N$5: D2.A, D3.C, R6.2, R7.1
- removed net VOUT: C6.1, D5.C
- new net +3V3: C2.+, C4.1, C5.1, D2.C, D6.C, IC1.VOUT, JP2.1, JP3.1, MDL2.VCC, R7.2, R8.1, R9.1, RN3A.1, RN3B.2, RN3C.2, U1.VDD
- new net +5V: C1.+, C6.1, D5.C, IC1.VIN, JP2.3, JP3.3, JP5.2, JP6.2
- new net CH_PD: MDL2.CH_PD, R8.2
- new net D1: RN3A.2, RN6C.2, U1.DATA
- new net D2: RN6D.2
- new net D5: D2.A, D3.C, MDL2.GPIO14, R6.2, R7.1
- new net DTR: JP4.1, Q4.E, R10.2
- new net GPIO0: MDL2.GPIO0, Q4.C, RN3B.1
- new net GPIO15: MDL2.GPIO15, RN3D.1
- new net GPIO2: MDL2.GPIO2, RN3C.1
- new net N$10: MDL2.GPIO13
- new net N$11: MDL2.GPIO16
- new net N$12: MDL2.GPIO12
- new net N$14: MDL2.ADC
- new net N$16: RN2B.2
- new net N$17: J4-3.S, RN2C.1
- new net N$18: J3-2.S, JP2.2
- new net N$19: J4-4.S, RN2D.1
- new net N$20: J4-2.S, JP3.2
- new net N$21: RN2C.2
- new net N$22: RN2D.2
- new net N$25: MDL2.GPIO5, RN6C.1
- new net N$27: D6.A, JP4.4
- new net N$30: MDL2.GPIO4, RN6D.1
- new net N$33: LED1.A, R18.1
- new net N$34: JP6.1, R18.2
- new net N$6: Q3.B, R10.1
- new net N$7: Q4.B, R11.1
- new net N$9: RN2A.2
- new net RST: MDL2.REST, Q3.E, R9.2, SW1.P, SW1.P1
- new net RTS: JP4.5, Q3.C, R11.2
- new net RX: MDL2.TXD, RN6A.1
- new net TX: MDL2.RXD, RN6B.1
- new net _RX: JP4.2, RN6A.2
- new net _TX: JP4.3, RN6B.2
- net GND: now also J3-1.S, J4-1.S, J5-1.S, JP1.GND, JP4.6, LED1.C, MDL2.GND, RN3D.2, SW1.S, SW1.S1; no longer C3.2, JP1.1
- net N$3: now also J3-3.S, RN2A.1; no longer C1.+, C3.1, IC1.VIN
- net N$4: now also J3-4.S, RN2B.1; no longer U1.DATA
- net VIN: now also J5-2.S, JP1.VCC, JP5.1; no longer JP1.2
Other:
- note added: "FDTI"
- note added: "Microcontrolador ESP8266"
- note added: "Sensor de Chuva"

Commit message: Prototype BOM
Parts:
- C4, C5: value (none) -> 100nF
- R10, R11, RN2: value (none) -> 1k
- R18, R7, R8, R9: value (none) -> 10k
- R3: value 0R -> 100R
- R6: value (none) -> 100R
Changed lines of the file:
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@@
 <part name="C2" library="wes" deviceset="CPOL-EU" device="C"/>
 <part name="GND1" library="SparkFun-Aesthetics" deviceset="GND" device=""/>
-<part name="C4" library="wes" deviceset="C-EU" device="C0805"/>
+<part name="C4" library="wes" deviceset="C-EU" device="C0805" value="100nF"/>
 <part name="U1" library="RHT03_DHT-22_AM2302" deviceset="RHT03_DHT-22_AM2302" device="RA"/>
 <part name="SUPPLY1" library="SparkFun-Aesthetics" deviceset="3.3V" device=""/>
-<part name="C5" library="wes" deviceset="C-EU" device="C0805"/>
+<part name="C5" library="wes" deviceset="C-EU" device="C0805" value="100nF"/>
 <part name="SUPPLY2" library="SparkFun-Aesthetics" deviceset="3.3V" device=""/>
 <part name="GND2" library="SparkFun-Aesthetics" deviceset="GND" device=""/>
@@
 <part name="D5" library="SparkFun-DiscreteSemi" deviceset="DIODE" device="SMA" value="DB2S31600"/>
 <part name="C7" library="wes" deviceset="C-EU" device="C0805" value="10uF 10V"/>
-<part name="R3" library="wes" deviceset="R-EU_" device="R0805" value="0R"/>
+<part name="R3" library="wes" deviceset="R-EU_" device="R0805" value="100R"/>
 <part name="Q2" library="SparkFun-DiscreteSemi" deviceset="MOSFET-NCHANNEL" device="BSS123LT1G" value="NFET"/>
 <part name="R5" library="wes" deviceset="R-EU_" device="R0805" value="100R"/>
@@
 <part name="U$1" library="lib_pluvion" deviceset="DRV5023FAQDBZR" device=""/>
 <part name="SUPPLY4" library="SparkFun-Aesthetics" deviceset="VIN" device=""/>
-<part name="R6" library="wes" deviceset="R-EU_" device="R0805"/>
-<part name="R7" library="wes" deviceset="R-EU_" device="R0805"/>
+<part name="R6" library="wes" deviceset="R-EU_" device="R0805" value="100R"/>
+<part name="R7" library="wes" deviceset="R-EU_" device="R0805" value="10k"/>
 <part name="SUPPLY5" library="SparkFun-Aesthetics" deviceset="3.3V" device=""/>
 <part name="D2" library="SparkFun-DiscreteSemi" deviceset="DIODE" device="SOD"/>
@@
 <part name="Q4" library="semicon-smd-ipc" deviceset="NPN-TRANSISTOR_" device="SOT23" value="S8050"/>
 <part name="+3V4" library="supply1" deviceset="+3V3" device=""/>
-<part name="R8" library="wes" deviceset="R-EU_" device="R0805"/>
-<part name="R9" library="wes" deviceset="R-EU_" device="R0805"/>
+<part name="R8" library="wes" deviceset="R-EU_" device="R0805" value="10k"/>
+<part name="R9" library="wes" deviceset="R-EU_" device="R0805" value="10k"/>
 <part name="MDL2" library="ESP8266-ESP12E" deviceset="ESP8266-12E" device="ESP8266-ESP12E"/>
 <part name="GND10" library="SparkFun-Aesthetics" deviceset="GND" device=""/>
@@
 <part name="J3" library="con-molex" deviceset="22-?-04" device="05-7048"/>
 <part name="GND13" library="SparkFun-Aesthetics" deviceset="GND" device=""/>
-<part name="RN2" library="resistor-dil" deviceset="4R-N" device="0603-ARV"/>
+<part name="RN2" library="resistor-dil" deviceset="4R-N" device="0603-ARV" value="1k"/>
 <part name="J4" library="con-molex" deviceset="22-?-04" device="05-7048"/>
 <part name="GND15" library="SparkFun-Aesthetics" deviceset="GND" device=""/>
@@
 <part name="SUPPLY11" library="SparkFun-Aesthetics" deviceset="VIN" device=""/>
 <part name="LED1" library="SparkFun-LED" deviceset="LED" device="1206"/>
-<part name="R18" library="wes" deviceset="R-EU_" device="R0805"/>
+<part name="R18" library="wes" deviceset="R-EU_" device="R0805" value="10k"/>
 <part name="JP6" library="SparkFun-Passives" deviceset="JUMPER-2" device="SMD-NO"/>
 <part name="RN3" library="resistor-dil" deviceset="4R-N" device="0603-ARV" value="10K"/>
@@
 <part name="SUPPLY8" library="SparkFun-Aesthetics" deviceset="3.3V" device=""/>
 <part name="D6" library="SparkFun-DiscreteSemi" deviceset="DIODE" device="SMA" value="DB2S31600"/>
-<part name="R10" library="wes" deviceset="R-EU_" device="R0805"/>
-<part name="R11" library="wes" deviceset="R-EU_" device="R0805"/>
+<part name="R10" library="wes" deviceset="R-EU_" device="R0805" value="1k"/>
+<part name="R11" library="wes" deviceset="R-EU_" device="R0805" value="1k"/>
 </parts>
 <sheets>

Commit message: Pluvion 1 Rev C
Connections:
- net RST: now also Q3.C; no longer Q3.E
- net RTS: now also Q3.E; no longer Q3.C
Other:
- moved on the sheet: Q3
Changed lines of the file:
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@@
 <grid distance="0.1" unitdist="inch" unit="inch" style="lines" multiple="1" display="no" altdistance="0.01" altunitdist="inch" altunit="inch"/>
 <layers>
-<layer number="1" name="Top" color="4" fill="1" visible="yes" active="no"/>
-<layer number="2" name="Route2" color="1" fill="3" visible="yes" active="no"/>
-<layer number="3" name="Route3" color="4" fill="3" visible="yes" active="no"/>
-<layer number="4" name="Route4" color="1" fill="4" visible="yes" active="no"/>
-<layer number="5" name="Route5" color="4" fill="4" visible="yes" active="no"/>
-<layer number="6" name="Route6" color="1" fill="8" visible="yes" active="no"/>
-<layer number="7" name="Route7" color="4" fill="8" visible="yes" active="no"/>
-<layer number="8" name="Route8" color="1" fill="2" visible="yes" active="no"/>
-<layer number="9" name="Route9" color="4" fill="2" visible="yes" active="no"/>
-<layer number="10" name="Route10" color="1" fill="7" visible="yes" active="no"/>
-<layer number="11" name="Route11" color="4" fill="7" visible="yes" active="no"/>
-<layer number="12" name="Route12" color="1" fill="5" visible="yes" active="no"/>
-<layer number="13" name="Route13" color="4" fill="5" visible="yes" active="no"/>
-<layer number="14" name="Route14" color="1" fill="6" visible="yes" active="no"/>
-<layer number="15" name="Route15" color="4" fill="6" visible="yes" active="no"/>
-<layer number="16" name="Bottom" color="1" fill="1" visible="yes" active="no"/>
-<layer number="17" name="Pads" color="2" fill="1" visible="yes" active="no"/>
-<layer number="18" name="Vias" color="2" fill="1" visible="yes" active="no"/>
-<layer number="19" name="Unrouted" color="6" fill="1" visible="yes" active="no"/>
-<layer number="20" name="Dimension" color="15" fill="1" visible="yes" active="no"/>
-<layer number="21" name="tPlace" color="7" fill="1" visible="yes" active="no"/>
-<layer number="22" name="bPlace" color="7" fill="1" visible="yes" active="no"/>
-<layer number="23" name="tOrigins" color="15" fill="1" visible="yes" active="no"/>
-<layer number="24" name="bOrigins" color="15" fill="1" visible="yes" active="no"/>
-<layer number="25" name="tNames" color="7" fill="1" visible="yes" active="no"/>
-<layer number="26" name="bNames" color="7" fill="1" visible="yes" active="no"/>
-<layer number="27" name="tValues" color="7" fill="1" visible="yes" active="no"/>
-<layer number="28" name="bValues" color="7" fill="1" visible="yes" active="no"/>
+<layer number="1" name="Top" color="4" fill="1" visible="no" active="no"/>
+<layer number="2" name="Route2" color="1" fill="3" visible="no" active="no"/>
+<layer number="3" name="Route3" color="4" fill="3" visible="no" active="no"/>
+<layer number="4" name="Route4" color="1" fill="4" visible="no" active="no"/>
+<layer number="5" name="Route5" color="4" fill="4" visible="no" active="no"/>
+<layer number="6" name="Route6" color="1" fill="8" visible="no" active="no"/>
+<layer number="7" name="Route7" color="4" fill="8" visible="no" active="no"/>
+<layer number="8" name="Route8" color="1" fill="2" visible="no" active="no"/>
+<layer number="9" name="Route9" color="4" fill="2" visible="no" active="no"/>
+<layer number="10" name="Route10" color="1" fill="7" visible="no" active="no"/>
+<layer number="11" name="Route11" color="4" fill="7" visible="no" active="no"/>
+<layer number="12" name="Route12" color="1" fill="5" visible="no" active="no"/>
+<layer number="13" name="Route13" color="4" fill="5" visible="no" active="no"/>
+<layer number="14" name="Route14" color="1" fill="6" visible="no" active="no"/>
+<layer number="15" name="Route15" color="4" fill="6" visible="no" active="no"/>
+<layer number="16" name="Bottom" color="1" fill="1" visible="no" active="no"/>
+<layer number="17" name="Pads" color="2" fill="1" visible="no" active="no"/>
+<layer number="18" name="Vias" color="2" fill="1" visible="no" active="no"/>
+<layer number="19" name="Unrouted" color="6" fill="1" visible="no" active="no"/>
+<layer number="20" name="Dimension" color="15" fill="1" visible="no" active="no"/>
+<layer number="21" name="tPlace" color="7" fill="1" visible="no" active="no"/>
+<layer number="22" name="bPlace" color="7" fill="1" visible="no" active="no"/>
+<layer number="23" name="tOrigins" color="15" fill="1" visible="no" active="no"/>
+<layer number="24" name="bOrigins" color="15" fill="1" visible="no" active="no"/>
+<layer number="25" name="tNames" color="7" fill="1" visible="no" active="no"/>
+<layer number="26" name="bNames" color="7" fill="1" visible="no" active="no"/>
+<layer number="27" name="tValues" color="7" fill="1" visible="no" active="no"/>
+<layer number="28" name="bValues" color="7" fill="1" visible="no" active="no"/>
 <layer number="29" name="tStop" color="7" fill="3" visible="no" active="no"/>
 <layer number="30" name="bStop" color="7" fill="6" visible="no" active="no"/>
@@
 <layer number="35" name="tGlue" color="7" fill="4" visible="no" active="no"/>
 <layer number="36" name="bGlue" color="7" fill="5" visible="no" active="no"/>
-<layer number="37" name="tTest" color="7" fill="1" visible="yes" active="no"/>
-<layer number="38" name="bTest" color="7" fill="1" visible="yes" active="no"/>
+<layer number="37" name="tTest" color="7" fill="1" visible="no" active="no"/>
+<layer number="38" name="bTest" color="7" fill="1" visible="no" active="no"/>
 <layer number="39" name="tKeepout" color="4" fill="11" visible="no" active="no"/>
 <layer number="40" name="bKeepout" color="1" fill="11" visible="no" active="no"/>
@@
 <layer number="44" name="Drills" color="7" fill="1" visible="no" active="no"/>
 <layer number="45" name="Holes" color="7" fill="1" visible="no" active="no"/>
-<layer number="46" name="Milling" color="3" fill="1" visible="yes" active="no"/>
-<layer number="47" name="Measures" color="7" fill="1" visible="yes" active="no"/>
-<layer number="48" name="Document" color="7" fill="1" visible="yes" active="no"/>
-<layer number="49" name="Reference" color="7" fill="1" visible="yes" active="no"/>
-<layer number="50" name="dxf" color="7" fill="1" visible="yes" active="no"/>
-<layer number="51" name="tDocu" color="7" fill="1" visible="yes" active="no"/>
-<layer number="52" name="bDocu" color="7" fill="1" visible="yes" active="no"/>
-<layer number="53" name="tGND_GNDA" color="7" fill="9" visible="yes" active="no"/>
-<layer number="54" name="bGND_GNDA" color="1" fill="9" visible="yes" active="no"/>
-<layer number="56" name="wert" color="7" fill="1" visible="yes" active="no"/>
-<layer number="57" name="tCAD" color="7" fill="1" visible="yes" active="no"/>
+<layer number="46" name="Milling" color="3" fill="1" visible="no" active="no"/>
+<layer number="47" name="Measures" color="7" fill="1" visible="no" active="no"/>
+<layer number="48" name="Document" color="7" fill="1" visible="no" active="no"/>
+<layer number="49" name="Reference" color="7" fill="1" visible="no" active="no"/>
+<layer number="50" name="dxf" color="7" fill="1" visible="no" active="no"/>
+<layer number="51" name="tDocu" color="7" fill="1" visible="no" active="no"/>
+<layer number="52" name="bDocu" color="7" fill="1" visible="no" active="no"/>
+<layer number="53" name="tGND_GNDA" color="7" fill="9" visible="no" active="no"/>
+<layer number="54" name="bGND_GNDA" color="1" fill="9" visible="no" active="no"/>
+<layer number="56" name="wert" color="7" fill="1" visible="no" active="no"/>
+<layer number="57" name="tCAD" color="7" fill="1" visible="no" active="no"/>
 <layer number="90" name="Modules" color="5" fill="1" visible="yes" active="yes"/>
 <layer number="91" name="Nets" color="2" fill="1" visible="yes" active="yes"/>
@@
 <instance part="SW1" gate="1" x="20.32" y="43.18" rot="MR0"/>
 <instance part="GND7" gate="1" x="10.16" y="35.56"/>
-<instance part="Q3" gate="G$1" x="22.86" y="-60.96" rot="R180"/>
+<instance part="Q3" gate="G$1" x="22.86" y="-60.96" rot="MR0"/>
 <instance part="Q4" gate="G$1" x="22.86" y="-81.28" rot="R180"/>
 <instance part="+3V4" gate="G$1" x="-43.18" y="33.02"/>
@@
 <net name="RST" class="0">
 <segment>
-<pinref part="Q3" gate="G$1" pin="E"/>
-<wire x1="20.32" y1="-55.88" x2="20.32" y2="-50.8" width="0.1524" layer="91"/>
 <wire x1="20.32" y1="-50.8" x2="35.56" y2="-50.8" width="0.1524" layer="91"/>
 <label x="35.56" y="-50.8" size="1.27" layer="95" xref="yes"/>
+<pinref part="Q3" gate="G$1" pin="C"/>
+<wire x1="20.32" y1="-55.88" x2="20.32" y2="-50.8" width="0.1524" layer="91"/>
 </segment>
 <segment>
@@
 <segment>
 <wire x1="40.64" y1="-81.28" x2="55.88" y2="-81.28" width="0.1524" layer="91"/>
-<pinref part="Q3" gate="G$1" pin="C"/>
 <wire x1="55.88" y1="-81.28" x2="71.12" y2="-81.28" width="0.1524" layer="91"/>
-<wire x1="20.32" y1="-66.04" x2="20.32" y2="-68.58" width="0.1524" layer="91"/>
 <wire x1="20.32" y1="-68.58" x2="55.88" y2="-68.58" width="0.1524" layer="91"/>
 <wire x1="55.88" y1="-68.58" x2="55.88" y2="-81.28" width="0.1524" layer="91"/>
@@
 <label x="71.12" y="-81.28" size="1.778" layer="95"/>
 <pinref part="R11" gate="G$1" pin="2"/>
-</segment>
-<segment>
+<pinref part="Q3" gate="G$1" pin="E"/>
+<wire x1="20.32" y1="-66.04" x2="20.32" y2="-68.58" width="0.1524" layer="91"/>
+</segment>
+<segment>
