File: Eletrônica/Principal/pluvionV0.brd (EAGLE design)
At the start: 47.3 x 80 mm, 12 parts, among them IC1 LD117AS33TR, SW1 Reset, U1 DHT22

Commit message: Update schematic
Parts:
- added DTR, GND_, RTS, RX, TX: LSP10, solpad:LSP10
- added Q1, Q2: S8050, semicon-smd-ipc:SOT23
- added R1, R3: 470R, rcl:M1206
- added R10, R4, R5, R6, R7, R8, R9: 10K, rcl:M1206
Connections:
- removed net N$4: ESP8266.9, SW1.1
- new net CH_PD: ESP8266.11, R6.2
- new net DTR: DTR.MP, Q2.2, R4.2
- new net GPIO0: ESP8266.4, Q2.3, R8.2
- new net GPIO15: ESP8266.2, R10.2
- new net GPIO2: ESP8266.3, R9.2
- new net N$10: ESP8266.15
- new net N$11: ESP8266.12
- new net N$12: ESP8266.14
- new net N$14: ESP8266.10
- new net N$3: R1.1, RX.MP
- new net N$5: R3.1, TX.MP
- new net N$6: Q1.1, R4.1
- new net N$7: Q2.1, R5.1
- new net N$9: ESP8266.5
- new net RST: ESP8266.9, Q1.2, R7.2, SW1.1
- new net RTS: Q1.3, R5.2, RTS.MP
- new net RX: ESP8266.8, R1.2
- new net TX: ESP8266.7, R3.2
- net +3V3: now also ESP8266.16, R6.1, R7.1, R8.1, R9.1
- net D3: no longer ESP8266.4
- net GNDA: now also GND_.MP, R10.1
Routing:
- net RST: track 0.00 -> 4.70 mm
- net N$4: track 4.70 -> 0.00 mm
Changed lines of the file:
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@@
 <element name="IC1" library="v-reg" package="SOT223" value="LD117AS33TR" x="-18.415" y="-2.54"/>
 <element name="HALL1" library="lib_pluvion" package="SOT23" value="DRV5023FAQDBZR" x="-19.05" y="-10.795"/>
+<element name="RX" library="solpad" package="LSP10" value="LSP10" x="-19.685" y="-17.78"/>
+<element name="TX" library="solpad" package="LSP10" value="LSP10" x="-19.685" y="-22.225"/>
+<element name="RTS" library="solpad" package="LSP10" value="LSP10" x="-19.685" y="-26.67"/>
+<element name="DTR" library="solpad" package="LSP10" value="LSP10" x="-19.685" y="-31.115"/>
+<element name="GND_" library="solpad" package="LSP10" value="LSP10" x="-19.685" y="-35.56"/>
+<element name="R1" library="rcl" package="M1206" value="470R" x="-19.05" y="-40.005"/>
+<element name="R3" library="rcl" package="M1206" value="470R" x="-19.05" y="-46.355"/>
+<element name="Q1" library="semicon-smd-ipc" package="SOT23" value="S8050" x="-19.05" y="-53.34"/>
+<element name="Q2" library="semicon-smd-ipc" package="SOT23" value="S8050" x="-19.05" y="-59.055"/>
+<element name="R4" library="rcl" package="M1206" value="10K" x="-19.05" y="-66.04"/>
+<element name="R5" library="rcl" package="M1206" value="10K" x="-19.05" y="-72.39"/>
+<element name="R6" library="rcl" package="M1206" value="10K" x="-19.05" y="-78.74"/>
+<element name="R7" library="rcl" package="M1206" value="10K" x="-19.05" y="-85.09"/>
+<element name="R8" library="rcl" package="M1206" value="10K" x="-19.05" y="-91.44"/>
+<element name="R9" library="rcl" package="M1206" value="10K" x="-19.05" y="-97.79"/>
+<element name="R10" library="rcl" package="M1206" value="10K" x="-19.05" y="-104.14"/>
 </elements>
 <signals>
@@
 <wire x1="5.715" y1="4.445" x2="9.62" y2="4.445" width="0.8128" layer="1"/>
 <contactref element="IC1" pad="4"/>
-<wire x1="31.75" y1="4.30231875" x2="35.35099375" y2="12.407171875" width="0" layer="19" extent="1-1"/>
-<wire x1="-18.415" y1="0.61" x2="5.08" y2="5.08" width="0" layer="19" extent="1-1"/>
+<contactref element="ESP8266" pad="16"/>
+<contactref element="R9" pad="1"/>
+<contactref element="R8" pad="1"/>
+<contactref element="R7" pad="1"/>
+<contactref element="R6" pad="1"/>
+<wire x1="-20.45" y1="-91.44" x2="-20.45" y2="-97.79" width="0" layer="19" extent="1-1"/>
+<wire x1="-20.45" y1="-85.09" x2="-20.45" y2="-91.44" width="0" layer="19" extent="1-1"/>
+<wire x1="-20.45" y1="-78.74" x2="-20.45" y2="-85.09" width="0" layer="19" extent="1-1"/>
+<wire x1="-18.415" y1="0.61" x2="-20.45" y2="-78.74" width="0" layer="19" extent="1-1"/>
+<wire x1="5.08" y1="5.08" x2="-18.415" y2="0.61" width="0" layer="19" extent="1-1"/>
+<wire x1="8.89" y1="4.54" x2="9.525" y2="4.54" width="0" layer="19" extent="1-1"/>
+<wire x1="35.35099375" y1="12.407171875" x2="31.75" y2="4.30231875" width="0" layer="19" extent="1-1"/>
 </signal>
 <signal name="GND">
@@
 <wire x1="-20.715" y1="-5.69" x2="2.8194" y2="22.1488" width="0" layer="19" extent="1-1"/>
 </signal>
-<signal name="N$4">
+<signal name="RST">
 <contactref element="ESP8266" pad="9"/>
 <contactref element="SW1" pad="1"/>
@@
 <wire x1="7.62" y1="19.05" x2="8.38" y2="19.05" width="0.6096" layer="1"/>
 <wire x1="8.38" y1="19.05" x2="8.89" y2="18.54" width="0.6096" layer="1"/>
+<contactref element="Q1" pad="2"/>
+<contactref element="R7" pad="2"/>
+<wire x1="-18.1" y1="-54.44" x2="-17.65" y2="-85.09" width="0" layer="19" extent="1-1"/>
+<wire x1="8.89" y1="18.54" x2="-18.1" y2="-54.44" width="0" layer="19" extent="1-1"/>
 </signal>
 <signal name="VCC/2">
@@
 </signal>
 <signal name="D3">
-<contactref element="ESP8266" pad="4"/>
 <contactref element="R2" pad="2"/>
 <contactref element="U1" pad="DATA"/>
@@
 <wire x1="27.94" y1="22.86" x2="27.94" y2="18.460503125" width="0.8128" layer="1"/>
 <wire x1="27.94" y1="18.460503125" x2="29.380034375" y2="17.02046875" width="0.8128" layer="1"/>
-<wire x1="25.09" y1="10.54" x2="26.899565625" y2="14.54" width="0" layer="19" extent="1-1"/>
 </signal>
 <signal name="D2">
@@
 <signal name="GNDA">
 <contactref element="HALL1" pad="3"/>
+<contactref element="GND_" pad="MP"/>
+<contactref element="R10" pad="1"/>
+<wire x1="-19.685" y1="-35.56" x2="-20.45" y2="-104.14" width="0" layer="19" extent="1-1"/>
+<wire x1="-19.05" y1="-9.695" x2="-19.685" y2="-35.56" width="0" layer="19" extent="1-1"/>
 </signal>
 <signal name="N$1">
@@
 <contactref element="HALL1" pad="1"/>
 </signal>
+<signal name="N$3">
+<contactref element="RX" pad="MP"/>
+<contactref element="R1" pad="1"/>
+<wire x1="-19.685" y1="-17.78" x2="-20.45" y2="-40.005" width="0" layer="19" extent="1-1"/>
+</signal>
+<signal name="N$5">
+<contactref element="TX" pad="MP"/>
+<contactref element="R3" pad="1"/>
+<wire x1="-19.685" y1="-22.225" x2="-20.45" y2="-46.355" width="0" layer="19" extent="1-1"/>
+</signal>
+<signal name="RX">
+<contactref element="R1" pad="2"/>
+<contactref element="ESP8266" pad="8"/>
+<wire x1="25.09" y1="18.54" x2="-17.65" y2="-40.005" width="0" layer="19" extent="1-1"/>
+</signal>
+<signal name="TX">
+<contactref element="R3" pad="2"/>
+<contactref element="ESP8266" pad="7"/>
+<wire x1="25.09" y1="16.54" x2="-17.65" y2="-46.355" width="0" layer="19" extent="1-1"/>
+</signal>
+<signal name="N$6">
+<contactref element="Q1" pad="1"/>
+<contactref element="R4" pad="1"/>
+<wire x1="-20" y1="-54.44" x2="-20.45" y2="-66.04" width="0" layer="19" extent="1-1"/>
+</signal>
+<signal name="N$7">
+<contactref element="R5" pad="1"/>
+<contactref element="Q2" pad="1"/>
+<wire x1="-20" y1="-60.155" x2="-20.45" y2="-72.39" width="0" layer="19" extent="1-1"/>
+</signal>
+<signal name="GPIO0">
+<contactref element="ESP8266" pad="4"/>
+<contactref element="Q2" pad="3"/>
+<contactref element="R8" pad="2"/>
+<wire x1="-19.05" y1="-57.955" x2="-17.65" y2="-91.44" width="0" layer="19" extent="1-1"/>
+<wire x1="25.09" y1="10.54" x2="-19.05" y2="-57.955" width="0" layer="19" extent="1-1"/>
+</signal>
+<signal name="RTS">
+<contactref element="RTS" pad="MP"/>
+<contactref element="R5" pad="2"/>
+<contactref element="Q1" pad="3"/>
+<wire x1="-19.05" y1="-52.24" x2="-17.65" y2="-72.39" width="0" layer="19" extent="1-1"/>
+<wire x1="-19.685" y1="-26.67" x2="-19.05" y2="-52.24" width="0" layer="19" extent="1-1"/>
+</signal>
+<signal name="DTR">
+<contactref element="DTR" pad="MP"/>
+<contactref element="R4" pad="2"/>
+<contactref element="Q2" pad="2"/>
+<wire x1="-18.1" y1="-60.155" x2="-17.65" y2="-66.04" width="0" layer="19" extent="1-1"/>
+<wire x1="-19.685" y1="-31.115" x2="-18.1" y2="-60.155" width="0" layer="19" extent="1-1"/>
+</signal>
+<signal name="CH_PD">
+<contactref element="R6" pad="2"/>
+<contactref element="ESP8266" pad="11"/>
+<wire x1="8.89" y1="14.54" x2="-17.65" y2="-78.74" width="0" layer="19" extent="1-1"/>
+</signal>
+<signal name="GPIO2">
+<contactref element="R9" pad="2"/>
+<contactref element="ESP8266" pad="3"/>
+<wire x1="25.09" y1="8.54" x2="-17.65" y2="-97.79" width="0" layer="19" extent="1-1"/>
+</signal>
+<signal name="GPIO15">
+<contactref element="R10" pad="2"/>
+<contactref element="ESP8266" pad="2"/>
+<wire x1="25.09" y1="6.54" x2="-17.65" y2="-104.14" width="0" layer="19" extent="1-1"/>
+</signal>
+<signal name="N$9">
+<contactref element="ESP8266" pad="5"/>
+</signal>
+<signal name="N$10">
+<contactref element="ESP8266" pad="15"/>
+</signal>
+<signal name="N$11">
+<contactref element="ESP8266" pad="12"/>
+</signal>
+<signal name="N$12">
+<contactref element="ESP8266" pad="14"/>
+</signal>
+<signal name="N$14">
+<contactref element="ESP8266" pad="10"/>
+</signal>
 </signals>

Commit message: Pluvion 1 Rev C
Connections:
- net RST: now also Q1.3; no longer Q1.2
- net RTS: now also Q1.2; no longer Q1.3
Changed lines of the file:
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@@
 <?xml version="1.0" encoding="utf-8"?>
 <!DOCTYPE eagle SYSTEM "eagle.dtd">
-<eagle version="7.6.0">
+<eagle version="7.3.0">
 <drawing>
 <settings>
@@
 <wire x1="7.62" y1="19.05" x2="8.38" y2="19.05" width="0.6096" layer="1"/>
 <wire x1="8.38" y1="19.05" x2="8.89" y2="18.54" width="0.6096" layer="1"/>
-<contactref element="Q1" pad="2"/>
 <contactref element="R7" pad="2"/>
-<wire x1="-18.1" y1="-54.44" x2="-17.65" y2="-85.09" width="0" layer="19" extent="1-1"/>
-<wire x1="8.89" y1="18.54" x2="-18.1" y2="-54.44" width="0" layer="19" extent="1-1"/>
+<contactref element="Q1" pad="3"/>
+<wire x1="-19.05" y1="-52.24" x2="-17.65" y2="-85.09" width="0" layer="19" extent="1-1"/>
+<wire x1="8.89" y1="18.54" x2="-19.05" y2="-52.24" width="0" layer="19" extent="1-1"/>
 </signal>
 <signal name="VCC/2">
@@
 <wire x1="25.09" y1="16.54" x2="-17.65" y2="-46.355" width="0" layer="19" extent="1-1"/>
 </signal>
-<signal name="N$6">
-<contactref element="Q1" pad="1"/>
-<contactref element="R4" pad="1"/>
-<wire x1="-20" y1="-54.44" x2="-20.45" y2="-66.04" width="0" layer="19" extent="1-1"/>
-</signal>
 <signal name="N$7">
 <contactref element="R5" pad="1"/>
@@
 <contactref element="RTS" pad="MP"/>
 <contactref element="R5" pad="2"/>
-<contactref element="Q1" pad="3"/>
-<wire x1="-19.05" y1="-52.24" x2="-17.65" y2="-72.39" width="0" layer="19" extent="1-1"/>
-<wire x1="-19.685" y1="-26.67" x2="-19.05" y2="-52.24" width="0" layer="19" extent="1-1"/>
+<contactref element="Q1" pad="2"/>
+<wire x1="-18.1" y1="-54.44" x2="-17.65" y2="-72.39" width="0" layer="19" extent="1-1"/>
+<wire x1="-19.685" y1="-26.67" x2="-18.1" y2="-54.44" width="0" layer="19" extent="1-1"/>
 </signal>
 <signal name="DTR">
@@
 <contactref element="ESP8266" pad="10"/>
 </signal>
+<signal name="N$4">
+<contactref element="R4" pad="1"/>
+<contactref element="Q1" pad="1"/>
+<wire x1="-20" y1="-54.44" x2="-20.45" y2="-66.04" width="0" layer="19" extent="1-1"/>
+</signal>
 </signals>
