File: Eletrônica/Principal/pluvionV0.sch (EAGLE design)
At the start: 12 parts, among them IC1 LD117AS33TR, SW1 Reset, U1 DHT22

Commit message: Update schematic
Parts:
- added DTR, GND_, RTS, RX, TX: LSP10, solpad:LSP10
- added Q1, Q2: S8050, semicon-smd-ipc:NPN-TRANSISTOR_SOT23
- added R1, R3: 470R, rcl:R-EU_M1206
- added R10, R4, R5, R6, R7, R8, R9: 10K, rcl:R-EU_M1206
Connections:
- removed net N$4: ESP8266.REST, SW1.S
- new net CH_PD: ESP8266.CH_PD, R6.2
- new net DTR: DTR.MP, Q2.E, R4.2
- new net GPIO0: ESP8266.GPIO0, Q2.C, R8.2
- new net GPIO15: ESP8266.GPIO15, R10.2
- new net GPIO2: ESP8266.GPIO2, R9.2
- new net N$10: ESP8266.GPIO13
- new net N$11: ESP8266.GPIO16
- new net N$12: ESP8266.GPIO12
- new net N$14: ESP8266.ADC
- new net N$3: R1.1, RX.MP
- new net N$5: R3.1, TX.MP
- new net N$6: Q1.B, R4.1
- new net N$7: Q2.B, R5.1
- new net N$9: ESP8266.GPIO5
- new net RST: ESP8266.REST, Q1.E, R7.2, SW1.S
- new net RTS: Q1.C, R5.2, RTS.MP
- new net RX: ESP8266.TXD, R1.2
- new net TX: ESP8266.RXD, R3.2
- net +3V3: now also ESP8266.VCC, R6.1, R7.1, R8.1, R9.1
- net D3: no longer ESP8266.GPIO0
- net GNDA: now also GND_.MP, R10.1
Other:
- note added: "FDTI"

Commit message: Pluvion 1 Rev C
Connections:
- net RST: now also Q1.C; no longer Q1.E
- net RTS: now also Q1.E; no longer Q1.C
Other:
- moved on the sheet: Q1
Changed lines of the file:
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@@
 <?xml version="1.0" encoding="utf-8"?>
 <!DOCTYPE eagle SYSTEM "eagle.dtd">
-<eagle version="7.6.0">
+<eagle version="7.3.0">
 <drawing>
 <settings>
@@
 <instance part="R3" gate="G$1" x="30.48" y="-27.94" rot="R90"/>
 <instance part="GND5" gate="1" x="66.04" y="-38.1"/>
-<instance part="Q1" gate="G$1" x="22.86" y="-60.96" rot="R180"/>
+<instance part="Q1" gate="G$1" x="22.86" y="-60.96" rot="MR0"/>
 <instance part="Q2" gate="G$1" x="22.86" y="-81.28" rot="R180"/>
 <instance part="R4" gate="G$1" x="35.56" y="-60.96"/>
@@
 </segment>
 <segment>
-<pinref part="Q1" gate="G$1" pin="E"/>
-<wire x1="20.32" y1="-55.88" x2="20.32" y2="-50.8" width="0.1524" layer="91"/>
 <wire x1="20.32" y1="-50.8" x2="35.56" y2="-50.8" width="0.1524" layer="91"/>
 <label x="35.56" y="-50.8" size="1.27" layer="95" xref="yes"/>
+<pinref part="Q1" gate="G$1" pin="C"/>
+<wire x1="20.32" y1="-55.88" x2="20.32" y2="-50.8" width="0.1524" layer="91"/>
 </segment>
 <segment>
@@
 </segment>
 </net>
-<net name="N$6" class="0">
-<segment>
-<pinref part="Q1" gate="G$1" pin="B"/>
-<pinref part="R4" gate="G$1" pin="1"/>
-<wire x1="25.4" y1="-60.96" x2="30.48" y2="-60.96" width="0.1524" layer="91"/>
-</segment>
-</net>
 <net name="N$7" class="0">
 <segment>
@@
 <pinref part="R5" gate="G$1" pin="2"/>
 <wire x1="40.64" y1="-81.28" x2="55.88" y2="-81.28" width="0.1524" layer="91"/>
-<pinref part="Q1" gate="G$1" pin="C"/>
 <wire x1="55.88" y1="-81.28" x2="71.12" y2="-81.28" width="0.1524" layer="91"/>
-<wire x1="20.32" y1="-66.04" x2="20.32" y2="-68.58" width="0.1524" layer="91"/>
 <wire x1="20.32" y1="-68.58" x2="55.88" y2="-68.58" width="0.1524" layer="91"/>
 <wire x1="55.88" y1="-68.58" x2="55.88" y2="-81.28" width="0.1524" layer="91"/>
 <junction x="55.88" y="-81.28"/>
+<pinref part="Q1" gate="G$1" pin="E"/>
+<wire x1="20.32" y1="-66.04" x2="20.32" y2="-68.58" width="0.1524" layer="91"/>
 </segment>
 </net>
@@
 </segment>
 </net>
+<net name="N$4" class="0">
+<segment>
+<pinref part="R4" gate="G$1" pin="1"/>
+<pinref part="Q1" gate="G$1" pin="B"/>
+<wire x1="30.48" y1="-60.96" x2="25.4" y2="-60.96" width="0.1524" layer="91"/>
+</segment>
+</net>
