File: Eletrônica/Principal/Pluvion 2.sch (EAGLE design)
At the start: 15 parts, among them Q1 PFET, Q2 NFET

Commit message: Pluvion V2
Parts:
- added R6: (no value), wes:R-EU_R0805
- added U1: (no value), RHT03_DHT-22_AM2302:RHT03_DHT-22_AM2302RA
Connections:
- new net N$17: R6.1, U1.DATA
- net +3V3: now also R6.2, U1.VDD
- net GND: now also U1.GND
Changed lines of the file:
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@@
 <part name="GND4" library="supply1" deviceset="GND" device=""/>
 <part name="GND5" library="supply1" deviceset="GND" device=""/>
+<part name="U1" library="RHT03_DHT-22_AM2302" deviceset="RHT03_DHT-22_AM2302" device="RA"/>
+<part name="GND6" library="supply1" deviceset="GND" device=""/>
+<part name="+3V2" library="supply1" deviceset="+3V3" device=""/>
+<part name="R6" library="wes" deviceset="R-EU_" device="R0805"/>
 </parts>
 <sheets>
@@
 <instance part="GND4" gate="1" x="101.6" y="147.32" rot="R90"/>
 <instance part="GND5" gate="1" x="101.6" y="129.54" rot="R90"/>
+<instance part="U1" gate="G$1" x="198.12" y="149.86"/>
+<instance part="GND6" gate="1" x="182.88" y="134.62"/>
+<instance part="+3V2" gate="G$1" x="182.88" y="165.1"/>
+<instance part="R6" gate="G$1" x="170.18" y="154.94" smashed="yes" rot="R90">
+<attribute name="NAME" x="158.75" y="156.4386" size="1.778" layer="95"/>
+<attribute name="VALUE" x="158.75" y="154.178" size="1.778" layer="96"/>
+</instance>
 </instances>
 <busses>
@@
 <pinref part="GND5" gate="1" pin="GND"/>
 </segment>
+<segment>
+<pinref part="U1" gate="G$1" pin="GND"/>
+<pinref part="GND6" gate="1" pin="GND"/>
+<wire x1="187.96" y1="142.24" x2="182.88" y2="142.24" width="0.1524" layer="91"/>
+<wire x1="182.88" y1="142.24" x2="182.88" y2="137.16" width="0.1524" layer="91"/>
+</segment>
 </net>
 <net name="N$1" class="0">
@@
 <wire x1="121.92" y1="60.96" x2="104.14" y2="60.96" width="0.1524" layer="91"/>
 </segment>
+<segment>
+<pinref part="U1" gate="G$1" pin="VDD"/>
+<wire x1="187.96" y1="157.48" x2="182.88" y2="157.48" width="0.1524" layer="91"/>
+<wire x1="182.88" y1="157.48" x2="182.88" y2="162.56" width="0.1524" layer="91"/>
+<pinref part="+3V2" gate="G$1" pin="+3V3"/>
+<pinref part="R6" gate="G$1" pin="2"/>
+<wire x1="170.18" y1="160.02" x2="175.26" y2="160.02" width="0.1524" layer="91"/>
+<wire x1="175.26" y1="160.02" x2="175.26" y2="157.48" width="0.1524" layer="91"/>
+<wire x1="175.26" y1="157.48" x2="182.88" y2="157.48" width="0.1524" layer="91"/>
+</segment>
 </net>
 <net name="N$3" class="0">
@@
 </segment>
 </net>
+<net name="N$17" class="0">
+<segment>
+<pinref part="U1" gate="G$1" pin="DATA"/>
+<pinref part="R6" gate="G$1" pin="1"/>
+<wire x1="170.18" y1="149.86" x2="175.26" y2="149.86" width="0.1524" layer="91"/>
+<wire x1="175.26" y1="149.86" x2="175.26" y2="152.4" width="0.1524" layer="91"/>
+<wire x1="175.26" y1="152.4" x2="187.96" y2="152.4" width="0.1524" layer="91"/>
+<wire x1="170.18" y1="149.86" x2="162.56" y2="149.86" width="0.1524" layer="91"/>
+</segment>
+</net>

Commit message: Pluvion V2 ready for prototyping
Parts:
- added C1: 10uF 10V, wes:C-EUC0805
- added J1: 22-05-7028-02, con-molex:22-05-7028-02
- D1, D4: device SparkFun-DiscreteSemi:DIODESMB -> SparkFun-DiscreteSemi:DIODESOD
- D5: device SparkFun-DiscreteSemi:DIODESMB -> SparkFun-DiscreteSemi:DIODESMA
Connections:
- removed net N$14 (its old number): U$2.D8
- removed net N$17 (its old number): R6.1, U1.DATA
- removed net N$18: U$2.3V@2
- removed net N$33: U$2.VIN
- new net +5V: C6.1, D5.C, JP5.2, U$2.VIN
- new net DHT_DATA: R6.1, U$2.D6, U1.DATA
- net +3V3: now also C1.1, U$2.3V@2; no longer C6.1, D5.C, JP5.2
- net ARD_OFF: now also U$2.D7
- net GND: now also C1.2, J1-1.S; no longer U$2.G@3, U$2.G@4
- net HALL: now also U$2.D8
- net N$12: now also U$2.G@3; no longer U$2.D6
- net N$13: now also U$2.G@4; no longer U$2.D7
- net VIN: now also J1-2.S
Other:
- moved on the sheet: R6
