File: Eletrônica/Principal/Pluvion 2 - Rev A.sch (EAGLE design)
At the start: 19 parts, among them J1 22-05-7028-02, Q1 PFET, Q2 NFET

Commit message: Shield Update
Connections:
- net ARD_OFF: now also U$2.D6; no longer U$2.D7
- net DHT_DATA: now also U$2.D5; no longer U$2.D6
- net HALL: now also U$2.D7; no longer U$2.D8
- net N$11: now also U$2.D8; no longer U$2.D5
Changed lines of the file:
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@@
 </segment>
 <segment>
-<pinref part="U$2" gate="G$1" pin="D7"/>
-<wire x1="88.9" y1="139.7" x2="99.06" y2="139.7" width="0.1524" layer="91"/>
-<label x="99.06" y="139.7" size="1.27" layer="95" xref="yes"/>
+<pinref part="U$2" gate="G$1" pin="D6"/>
+<wire x1="88.9" y1="142.24" x2="99.06" y2="142.24" width="0.1524" layer="91"/>
+<label x="99.06" y="142.24" size="1.27" layer="95" xref="yes"/>
 </segment>
 </net>
@@
 </segment>
 <segment>
-<pinref part="U$2" gate="G$1" pin="D8"/>
-<wire x1="88.9" y1="137.16" x2="99.06" y2="137.16" width="0.1524" layer="91"/>
-<label x="99.06" y="137.16" size="1.27" layer="95" xref="yes"/>
+<pinref part="U$2" gate="G$1" pin="D7"/>
+<wire x1="88.9" y1="139.7" x2="99.06" y2="139.7" width="0.1524" layer="91"/>
+<label x="99.06" y="139.7" size="1.27" layer="95" xref="yes"/>
 </segment>
 </net>
@@
 <pinref part="U$2" gate="G$1" pin="D4"/>
 <wire x1="88.9" y1="152.4" x2="99.06" y2="152.4" width="0.1524" layer="91"/>
-</segment>
-</net>
-<net name="N$11" class="0">
-<segment>
-<pinref part="U$2" gate="G$1" pin="D5"/>
-<wire x1="88.9" y1="144.78" x2="99.06" y2="144.78" width="0.1524" layer="91"/>
 </segment>
 </net>
@@
 </segment>
 <segment>
-<pinref part="U$2" gate="G$1" pin="D6"/>
-<wire x1="88.9" y1="142.24" x2="99.06" y2="142.24" width="0.1524" layer="91"/>
-<label x="99.06" y="142.24" size="1.27" layer="95" xref="yes"/>
+<pinref part="U$2" gate="G$1" pin="D5"/>
+<wire x1="88.9" y1="144.78" x2="99.06" y2="144.78" width="0.1524" layer="91"/>
+<label x="99.06" y="144.78" size="1.27" layer="95" xref="yes"/>
 </segment>
 </net>
@@
 </segment>
 </net>
+<net name="N$11" class="0">
+<segment>
+<pinref part="U$2" gate="G$1" pin="D8"/>
+<wire x1="88.9" y1="137.16" x2="99.06" y2="137.16" width="0.1524" layer="91"/>
+</segment>
+</net>
