File: Eletrônica/Principal/Pluvion 2 - Rev B.sch (EAGLE design)
At the start: 19 parts, among them J1 22-05-7028-02, Q1 PFET, Q2 NFET

Commit message: Shield Update
Parts:
- added JP1: (no value), SparkFun-Passives:JUMPER-2PTH
- added R7: 10k, wes:R-EU_R0805
- R6: value (none) -> 10K
Connections:
- removed net N$17: U$2.3V
- new net +3VLEFT: JP1.1, U$2.3V
- net HALL: now also R7.2
- net VIN: now also JP1.2, R7.1
Changed lines of the file:
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@@
 <part name="GND6" library="supply1" deviceset="GND" device=""/>
 <part name="+3V2" library="supply1" deviceset="+3V3" device=""/>
-<part name="R6" library="wes" deviceset="R-EU_" device="R0805"/>
+<part name="R6" library="wes" deviceset="R-EU_" device="R0805" value="10K"/>
 <part name="P+1" library="supply1" deviceset="+5V" device=""/>
 <part name="P+2" library="supply1" deviceset="+5V" device=""/>
@@
 <part name="SUPPLY1" library="SparkFun-Aesthetics" deviceset="VIN" device=""/>
 <part name="GND8" library="supply1" deviceset="GND" device=""/>
+<part name="R7" library="wes" deviceset="R-EU_" device="R0805" value="10k"/>
+<part name="JP1" library="SparkFun-Passives" deviceset="JUMPER-2" device="PTH"/>
 </parts>
 <sheets>
@@
 </instance>
 <instance part="GND8" gate="1" x="17.78" y="55.88"/>
+<instance part="R7" gate="G$1" x="30.48" y="55.88" smashed="yes" rot="R270">
+<attribute name="NAME" x="34.29" y="54.8386" size="1.778" layer="95"/>
+<attribute name="VALUE" x="34.29" y="57.658" size="1.778" layer="96"/>
+</instance>
+<instance part="JP1" gate="A" x="-12.7" y="48.26"/>
 </instances>
 <busses>
@@
 <segment>
 <pinref part="U$1" gate="G$1" pin="VCC"/>
-<wire x1="20.32" y1="43.18" x2="25.4" y2="43.18" width="0.1524" layer="91"/>
+<wire x1="20.32" y1="43.18" x2="22.86" y2="43.18" width="0.1524" layer="91"/>
+<wire x1="22.86" y1="43.18" x2="25.4" y2="43.18" width="0.1524" layer="91"/>
 <wire x1="25.4" y1="43.18" x2="25.4" y2="45.72" width="0.1524" layer="91"/>
 <pinref part="SUPPLY4" gate="G$1" pin="VIN"/>
+<wire x1="22.86" y1="43.18" x2="22.86" y2="60.96" width="0.1524" layer="91"/>
+<junction x="22.86" y="43.18"/>
+<pinref part="R7" gate="G$1" pin="1"/>
+<wire x1="22.86" y1="60.96" x2="30.48" y2="60.96" width="0.1524" layer="91"/>
+<wire x1="20.32" y1="43.18" x2="20.32" y2="48.26" width="0.1524" layer="91"/>
+<junction x="20.32" y="43.18"/>
+<wire x1="20.32" y1="48.26" x2="-7.62" y2="48.26" width="0.1524" layer="91"/>
+<wire x1="-7.62" y1="48.26" x2="-7.62" y2="45.72" width="0.1524" layer="91"/>
+<pinref part="JP1" gate="A" pin="2"/>
+<wire x1="-7.62" y1="45.72" x2="-10.16" y2="45.72" width="0.1524" layer="91"/>
 </segment>
 <segment>
@@
 <junction x="30.48" y="40.64"/>
 <label x="35.56" y="17.78" size="1.27" layer="95" xref="yes"/>
+<pinref part="R7" gate="G$1" pin="2"/>
+<wire x1="30.48" y1="40.64" x2="30.48" y2="50.8" width="0.1524" layer="91"/>
 </segment>
 <segment>
@@
 </segment>
 </net>
-<net name="N$17" class="0">
+<net name="+3VLEFT" class="0">
 <segment>
 <pinref part="U$2" gate="G$1" pin="3V"/>
 <wire x1="55.88" y1="137.16" x2="48.26" y2="137.16" width="0.1524" layer="91"/>
-</segment>
-</net>
+<label x="38.1" y="137.16" size="1.778" layer="95" rot="R180"/>
+</segment>
+<segment>
+<pinref part="JP1" gate="A" pin="1"/>
+<wire x1="-12.7" y1="45.72" x2="-20.32" y2="45.72" width="0.1524" layer="91"/>
+<label x="-22.86" y="45.72" size="1.778" layer="95" rot="R180"/>
+</segment>
+</net>
