File: Eletrônica/Principal/Pluvion 2 - Rev C.brd (EAGLE design)
At the start: 34.3 x 67.5 mm, 19 parts, among them J1 22-05-7028-02, Q1 PFET, Q2 NFET

Commit message: Shield Update
Parts:
- moved U1 5.30 mm to (17.1, 31.5)
- moved R6 5.10 mm to (17.1, 29.2)
- moved C1 4.90 mm to (17.1, 26.9)
- moved D5 2.91 mm to (11.4, 9.23)
- moved D4 2.62 mm to (26.8, 14.5)
- moved R1 2.62 mm to (26.8, 9.43)
- moved R5 2.62 mm to (26.8, 12.0)
- moved Q2 2.40 mm to (18.4, 14.1)
- moved C6 2.40 mm to (6.03, 12.8)
- moved D1 2.40 mm to (10.8, 15.4)
- moved J1 2.40 mm to (3.17, 7.76)
- moved JP5 2.40 mm to (12.1, 5.22)
- moved Q1 2.40 mm to (18.4, 8.39)
- moved R2 2.40 mm to (10.8, 12.8)
- moved U$1 2.40 mm to (17.2, 5.30)
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Connections:
- net ARD_OFF: now also U$2.D6; no longer U$2.D7
- net DHT_DATA: now also U$2.D5; no longer U$2.D6
- net HALL: now also U$2.D7; no longer U$2.D8
- net N$11: now also U$2.D8; no longer U$2.D5
Routing:
- net +3V3: track 61.3 -> 28.4 mm
- net GND: track 0.00 -> 21.9 mm
- net +5V: track 11.3 -> 18.5 mm
- net HALL: track 24.7 -> 29.4 mm, vias 2 -> 1
- net DHT_DATA: track 26.9 -> 24.0 mm
- net ARD_OFF: track 43.6 -> 45.9 mm, vias 0 -> 1
- net N$1: track 11.5 -> 9.40 mm
- net VIN: track 32.7 -> 34.3 mm
- net N$8: track 5.19 -> 6.65 mm
- net BUTTONS: track 17.0 -> 18.4 mm
Other:
- board size 34.3 x 67.5 mm -> 34.3 x 58.9 mm
- board text added: ".ON"
- board text added: "PLUVI"
